File: hardware/pcb/v2.1/kicad/digits-pcb.kicad_pcb (KiCad board)
At the start: 2 copper layers, 76.2 x 61.9 mm, 71 parts, among them J1 Conn_02x20_Odd_Even, J3 VIN_BARREL_PIGTAIL, J4 Conn_01x07, J6 Conn_01x02, J7 Screw_Terminal_01x02, J8 Conn_01x04, J9 Conn_01x03, SW1 SW_Push, U1 LM2596S-5, U2 DRV8871DDAR, U3 RP2040, U4 W25Q16JVSSIQ, U5 AMS1117-3.3, U6 TLV320AIC3104IRHBR, U7 XC6206P182MR, Y1 ABM8-272-T3

Commit message: fix(hardware): swap V2.1 J6 pad numbers on footprint to match schematic
Complements the schematic-side J6 swap by updating the PCB footprint
instance directly: flips pad "1" and pad "2" labels on the two J6
pads (copper unchanged) so the PCB netlist agrees with the schematic
(pin 1 = GND, pin 2 = LED_A) without requiring a physical re-route
of the two short nets around J6.

DRC: 51 violations total, 1 more than V2's baseline of 50. The new
entry is a lib_footprint_mismatch on J6, expected: the footprint
instance no longer matches its library template because pad labels
differ. Same kind of "Local override; warning" as the six other
footprint-instance tweaks already on the board.
Connections:
- J6 pad 1: LED_A -> GND
- J6 pad 2: GND -> LED_A
Changed lines of the file:
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@@
 			)
 		)
-		(pad "1" smd roundrect
+		(pad "2" smd roundrect
 			(at -0.75 0.7 90)
 			(size 0.7 3.7)
@@
 			(roundrect_rratio 0.25)
 			(net "LED_A")
-			(pinfunction "Pin_1_1")
+			(pinfunction "Pin_2_2")
 			(pintype "passive")
 		)
-		(pad "2" smd roundrect
+		(pad "1" smd roundrect
 			(at 0.75 0.7 90)
 			(size 0.7 3.7)
@@
 			(roundrect_rratio 0.25)
 			(net "GND")
-			(pinfunction "Pin_2_2")
+			(pinfunction "Pin_1_1")
 			(pintype "passive")
 		)
